Commit message: required changes to upgrade to noetic

File: urdf/web-diff_drive_urdf.xacro (robot description, xacro)
@@ -56,4 +56,11 @@
 <!-- ////////////////////////////////////////////////////////////-->
 <!-- chassis-->
+ <link name="dummy_link">
+      <visual>
+        <geometry>
+          <sphere radius="0.001"/>
+        </geometry>
+      </visual>
+ </link>
  <link name="chassis">
     <visual>
@@ -71,4 +78,9 @@
    <xacro:inertial_matrix mass="5.0"/>
  </link>
+ <joint name="dummy_joint" type="fixed">
+    <origin xyz="0 0 0"/>
+    <parent link="dummy_link"/>
+    <child link="chassis"/>
+ </joint>
  <gazebo reference="chassis">
     <turnGravityOff>false</turnGravityOff>
